File: Detection_V1_PCB/492pcb/Sensor_Functions_Project_06.kicad_sch (KiCad schematic)
At the start: 7 parts, among them J14 Conn_02x05_Odd_Even, U2 BME680, U4 SCD40-D-R2

Commit message: a
Parts:
- renumbered J14 to J8, U4 to U3
Changed lines of the file:
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@@
+				)
+			)
+			(project "Processor_Schematic_Project_06"
+				(path "/7cd6380d-12c8-4529-8126-c1d91df0fbc9/19d3cce4-1283-4e98-b8c5-4082ee9eca09"
+					(reference "U2")
+					(unit 1)
 				)
 			)
@@
 				)
 			)
+			(project "Processor_Schematic_Project_06"
+				(path "/7cd6380d-12c8-4529-8126-c1d91df0fbc9/19d3cce4-1283-4e98-b8c5-4082ee9eca09"
+					(reference "TP1")
+					(unit 1)
+				)
+			)
 		)
 	)
@@
 		(dnp no)
 		(fields_autoplaced yes)
-		(property "Reference" "#PWR013"
+		(property "Reference" "#PWR011"
 			(at 165.1 114.3 0)
 			(effects
@@
 				)
 			)
+			(project "Processor_Schematic_Project_06"
+				(path "/7cd6380d-12c8-4529-8126-c1d91df0fbc9/19d3cce4-1283-4e98-b8c5-4082ee9eca09"
+					(reference "#PWR011")
+					(unit 1)
+				)
+			)
 		)
 	)
@@
 				)
 			)
+			(project "Processor_Schematic_Project_06"
+				(path "/7cd6380d-12c8-4529-8126-c1d91df0fbc9/19d3cce4-1283-4e98-b8c5-4082ee9eca09"
+					(reference "TP2")
+					(unit 1)
+				)
+			)
 		)
 	)
@@
 		(dnp no)
 		(fields_autoplaced yes)
-		(property "Reference" "U4"
+		(property "Reference" "U3"
 			(at 156.21 99.0599 0)
 			(effects
@@
 				)
 			)
+			(project "Processor_Schematic_Project_06"
+				(path "/7cd6380d-12c8-4529-8126-c1d91df0fbc9/19d3cce4-1283-4e98-b8c5-4082ee9eca09"
+					(reference "U3")
+					(unit 1)
+				)
+			)
 		)
 	)
@@
 		(dnp no)
 		(fields_autoplaced yes)
-		(property "Reference" "#PWR04"
+		(property "Reference" "#PWR08"
 			(at 106.68 121.92 0)
 			(effects
@@
 				)
 			)
+			(project "Processor_Schematic_Project_06"
+				(path "/7cd6380d-12c8-4529-8126-c1d91df0fbc9/19d3cce4-1283-4e98-b8c5-4082ee9eca09"
+					(reference "#PWR08")
+					(unit 1)
+				)
+			)
 		)
 	)
@@
 				)
 			)
+			(project "Processor_Schematic_Project_06"
+				(path "/7cd6380d-12c8-4529-8126-c1d91df0fbc9/19d3cce4-1283-4e98-b8c5-4082ee9eca09"
+					(reference "TP3")
+					(unit 1)
+				)
+			)
 		)
 	)
@@
 		(on_board yes)
 		(dnp no)
-		(property "Reference" "J14"
+		(property "Reference" "J8"
 			(at 224.79 90.17 0)
 			(effects
@@
 				)
 			)
+			(project "Processor_Schematic_Project_06"
+				(path "/7cd6380d-12c8-4529-8126-c1d91df0fbc9/19d3cce4-1283-4e98-b8c5-4082ee9eca09"
+					(reference "J8")
+					(unit 1)
+				)
+			)
 		)
 	)
@@
 		(on_board yes)
 		(dnp no)
-		(property "Reference" "#PWR06"
+		(property "Reference" "#PWR010"
 			(at 127 81.28 0)
 			(effects
@@
 				)
 			)
+			(project "Processor_Schematic_Project_06"
+				(path "/7cd6380d-12c8-4529-8126-c1d91df0fbc9/19d3cce4-1283-4e98-b8c5-4082ee9eca09"
+					(reference "#PWR010")
+					(unit 1)
+				)
+			)
 		)
 	)
@@
 		(dnp no)
 		(fields_autoplaced yes)
-		(property "Reference" "#PWR014"
+		(property "Reference" "#PWR012"
 			(at 215.9 114.3 0)
 			(effects
@@
 				)
 			)
+			(project "Processor_Schematic_Project_06"
+				(path "/7cd6380d-12c8-4529-8126-c1d91df0fbc9/19d3cce4-1283-4e98-b8c5-4082ee9eca09"
+					(reference "#PWR012")
+					(unit 1)
+				)
+			)
 		)
 	)
@@
 		(dnp no)
 		(fields_autoplaced yes)
-		(property "Reference" "#PWR05"
+		(property "Reference" "#PWR09"
 			(at 111.76 121.92 0)
 			(effects
@@
 				)
 			)
+			(project "Processor_Schematic_Project_06"
+				(path "/7cd6380d-12c8-4529-8126-c1d91df0fbc9/19d3cce4-1283-4e98-b8c5-4082ee9eca09"
+					(reference "#PWR09")
+					(unit 1)
+				)
+			)
 		)
 	)
@@
 					(reference "TP4")
 					(unit 1)
+				)
+			)
+			(project "Processor_Schematic_Project_06"
+				(path "/7cd6380d-12c8-4529-8126-c1d91df0fbc9/19d3cce4-1283-4e98-b8c5-4082ee9eca09"
+					(reference "TP4")
+					(unit 1)
